File: esp8266/pcb/urc/urc.sch (KiCad schematic (older format))
At the start: 10 parts, among them T1 2N2222a

Commit message: committing changes
Parts:
- RGREEN1, RRED1: value R -> 820R
- RUP1: value R -> 4.7K
Changed lines of the file:
@@
 P 8450 5150
 F 0 "RGREEN1" H 8520 5196 50  0000 L CNN
-F 1 "R" H 8520 5105 50  0000 L CNN
+F 1 "820R" H 8520 5105 50  0000 L CNN
 F 2 "Resistor_THT:R_Axial_DIN0204_L3.6mm_D1.6mm_P2.54mm_Vertical" V 8380 5150 50  0001 C CNN
 F 3 "~" H 8450 5150 50  0001 C CNN
@@
 P 8850 5150
 F 0 "RRED1" H 8920 5196 50  0000 L CNN
-F 1 "R" H 8920 5105 50  0000 L CNN
+F 1 "820R" H 8920 5105 50  0000 L CNN
 F 2 "Resistor_THT:R_Axial_DIN0204_L3.6mm_D1.6mm_P2.54mm_Vertical" V 8780 5150 50  0001 C CNN
 F 3 "~" H 8850 5150 50  0001 C CNN
@@
 P 6350 3050
 F 0 "RUP1" H 6420 3096 50  0000 L CNN
-F 1 "R" H 6420 3005 50  0000 L CNN
+F 1 "4.7K" H 6420 3005 50  0000 L CNN
 F 2 "Resistor_THT:R_Axial_DIN0204_L3.6mm_D1.6mm_P2.54mm_Vertical" V 6280 3050 50  0001 C CNN
 F 3 "~" H 6350 3050 50  0001 C CNN
